File: sub_081/081_fotocellule.brd (EAGLE design)
At the start: 100 x 80 mm, 40 parts, among them IC1 TL082P, IC2 TL082P, IC3 LM555N, T1 BD647

Commit message: Risistemati i due progetti per l'utilizzo dei singoli/doppi opamp
Parts:
- removed LED+, LED+1, LED-, LED-1, PD+, PD+1, PD-, PD-1: WIREPAD2,54/1,0, wirepad:2,54/1,0
- added C4, C5, C6, C7: 4.7uF, resistor:E2,5-6
- added D1, D2, D3, D4: 1N4004, diode:DO41-10
- added IC10, IC4, IC5, IC6, IC7, IC8, IC9: TL081P, linear:DIL08
- added PAD10, PAD11, PAD12, PAD13, PAD14, PAD15, PAD16, PAD17, PAD18, PAD19, PAD2, PAD20, PAD3, PAD4, PAD6, PAD7, PAD8, PAD9: WIREPAD2,54/1,0, wirepad:2,54/1,0
- added Q1, Q2, Q3, Q4: 2N3904, transistor-npn:TO92
- added R23, R34, R45: 1.5k, resistor:0207/10
- added R24, R35, R46: 33, resistor:0207/10
- added R25, R36, R47: 330, resistor:0207/10
- added R26, R28, R29, R32, R33, R37, R39, R40, R43, R44, R48: 1k, resistor:0207/10
- added R27, R38: 1M, resistor:0207/10
- added R30, R41: 2.2 k, resistor:0207/10
- added R31, R42: 1 M, resistor:0207/10
- C1: value 4.7uF -> 100nF; device resistor:E2,5-6 -> resistor:C025-024X044
- C2: value 100nF -> 100 nF
- C3: value 4.7uF -> 100 nF; device resistor:E2,5-6 -> resistor:C025-024X044
- IC1: value TL082P -> 7805TV; device linear:DIL08 -> linear:TO220V
- IC2: value TL082P -> NE555N
- IC3: value LM555N -> TL081P
- R1: value 1M -> 470
- R10: value 4.7k -> 1 M
- R12: value 150 -> 1k
- R13: value (none) -> 1.5k
- R14: value 1M -> 330
- R16, R6: value 1k -> 1M
- R17: value 2.2 k -> 1k
- R18: value 1 M -> 1k
- R19: value 1k -> 2.2 k
- R2: value 1k -> 4.7k
- R20: value 1k -> 1 M
- R21, R8: value 1.5k -> 1k
- R22: value 33 -> 1k
- R4: value 2.2 k -> 150
- R5: value 1 M -> 33
- R9: value 33 -> 2.2 k
- moved R15 116.8 mm to (73.7, 55.9), turned to 180 degrees
- moved PAD1 99.4 mm to (61.0, 63.5)
- moved R14 98.3 mm to (74.9, 38.1), turned to 270 degrees
- moved IC2 66.0 mm to (15.2, 55.9), turned to 180 degrees
- moved IC3 52.9 mm to (62.2, 52.1)
- moved R12 52.5 mm to (50.8, 39.4), turned to 270 degrees
- moved LED1 49.0 mm to (3.81, 64.8), turned to 0 degrees
- moved C3 43.1 mm to (8.89, 38.1), turned to 180 degrees
- moved PAD5 43.1 mm to (78.7, 50.8)
- moved R13 42.7 mm to (53.3, 39.4), turned to 90 degrees
- moved T1 41.2 mm to (31.8, 63.5), turned to 270 degrees
- moved R11 41.0 mm to (61.0, 44.5), turned to 180 degrees
- moved R9 40.2 mm to (50.8, 50.8)
- moved R10 38.9 mm to (50.8, 55.9), turned to 0 degrees
- moved R5 33.1 mm to (50.8, 61.0)
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Connections:
- new net +5V: C3.1, IC1.3, IC10.7, IC2.8, IC3.7, IC4.7, IC5.7, IC6.7, IC7.7, IC8.7, IC9.7, LED1.A, PAD1.1, PAD13.1, PAD18.1, PAD8.1, R13.2, R15.2, R16.2, R2.2, R23.2, R26.2, R27.2, R34.2, R37.2, R38.2, R45.2, R48.2, R6.2
- new net N$25: PAD10.1, Q2.1, R26.1
- new net N$26: D2.C, Q2.2, R25.1
- new net N$27: IC6.6, R25.2
- new net N$28: PAD11.1, R27.1, R28.1
- new net N$29: IC7.2, R28.2, R31.1
- new net N$30: IC7.3, R29.2, R30.2
- new net N$31: IC7.6, R31.2, R32.1
- new net N$32: C6.+, IC8.2, R32.2
- new net N$33: IC8.3, R33.2, R34.1
- new net N$34: PAD14.1, R35.2
- new net N$36: PAD15.1, Q3.1, R37.1
- new net N$37: D3.C, Q3.2, R36.1
- new net N$38: IC8.6, R36.2
- new net N$39: PAD16.1, R38.1, R39.1
- new net N$40: IC9.2, R39.2, R42.1
- new net N$41: IC9.3, R40.2, R41.2
- new net N$42: IC9.6, R42.2, R43.1
- new net N$43: C7.+, IC10.2, R43.2
- new net N$44: IC10.3, R44.2, R45.1
- new net N$45: PAD19.1, R46.2
- new net N$46: R18.1, R24.1, R29.1, R35.1, R40.1, R46.1, R5.1, R7.1, T1.2
- new net N$47: PAD20.1, Q4.1, R48.1
- new net N$48: D4.C, Q4.2, R47.1
- new net N$49: IC10.6, R47.2
- net GND: now also C1.2, C3.2, C4.-, C5.-, C6.-, C7.-, D1.A, D2.A, D3.A, D4.A, IC1.2, IC10.4, IC2.1, IC3.4, IC4.4, IC5.4, IC6.4, IC7.4, IC8.4, IC9.4, PAD12.1, PAD17.1, PAD4.1, PAD7.1, Q1.3, Q2.3, Q3.3, Q4.3, R1.1, R12.1, R19.1, R22.1, R30.1, R33.1, R41.1, R44.1, R9.1; no longer C1.-, C3.-, IC1.4, IC2.4, IC3.1, PD-.1, PD-1.1, R13.1, R17.1, R20.1, R4.1, R7.1
- net N$1: now also PAD3.1, R6.1, R8.1; no longer PD+.1, R1.1, R2.1
- net N$10: now also C1.1, IC2.2, IC2.6, R3.1; no longer C2.1, IC3.2, IC3.6, R11.1
- net N$11: now also IC4.6, R14.2; no longer IC3.7, R10.1, R11.2
- net N$12: now also R4.2; no longer R12.2
- net N$13: now also IC5.2, R17.2, R20.1; no longer IC1.7, PAD5.1
- net N$14: now also R1.2; no longer R13.2
- net N$15: now also IC2.7, R2.1, R3.2; no longer PD+1.1, R14.1, R15.1
- net N$16: now also PAD5.1, Q1.1, R15.1; no longer IC2.2, R15.2, R18.1
- net N$17: now also IC5.3, R18.2, R19.2; no longer IC2.3, R16.2, R17.2
- net N$18: now also D1.C, Q1.2, R14.1; no longer IC2.1, R18.2, R19.1
- net N$19: now also IC5.6, R20.2, R21.1; no longer C3.+, IC2.6, R19.2
- net N$2: now also IC3.2, R10.1, R8.2; no longer IC1.2, R2.2, R5.1
- net N$20: now also C5.+, IC6.2, R21.2; no longer IC2.5, R20.2, R21.1
- net N$21: now also IC6.3, R23.1; no longer LED-1.1
- net N$23: now also PAD9.1, R24.2; no longer IC2.7, PAD1.1
- net N$3: now also IC3.3, R7.2, R9.2; no longer IC1.3, R3.2, R4.2
- net N$4: now also IC3.6, R10.2, R11.1; no longer IC1.1, R5.2, R6.1
- net N$5: now also C4.+, IC4.2, R11.2; no longer C1.+, IC1.6, R6.2
- net N$6: now also IC4.3, R12.2, R13.1; no longer IC1.5, R7.2, R8.1
- net N$7: now also PAD2.1, R5.2; no longer LED-.1, R9.2
- net N$8: now also PAD6.1, R17.1; no longer R22.1, R3.1, R9.1, T1.2
- net N$9: now also IC2.3, R4.1; no longer IC3.3, R12.1
- net VCC: now also C2.1, IC1.1; no longer IC1.8, IC2.8, IC3.8, LED+.1, LED+1.1, LED1.A, R1.2, R10.2, R14.2, R21.2, R8.2
Other:
- board size 100 x 80 mm -> 100 x 69.8 mm
