File: sub_082/fotocellule.brd (EAGLE design)
At the start: 100 x 69.8 mm, 39 parts, among them IC1 TL082P, IC3 NE555N, IC5 7805TV, IC6 NE555N, Q1 2N3904, T1 BD647

Commit message: Rewired correctly sub082
Parts:
- removed IC5: 7805TV, linear:TO220V
- removed IC6: NE555N, linear:DIL08
- removed OUT: WIREPAD2,54/1,0, wirepad:2,54/1,0
- removed R32: 56k, resistor:0207/10
- removed R33: 22k, resistor:0207/10
- removed R35: 470, resistor:0207/10
- added IC2: NE555N, linear:DIL08
- added IC4: TL082P, linear:DIL08
- added JP1: POWER_JACKPTH_LOCK, SparkFun-Connectors:POWER_JACK_PTH_LOCK
- added LEDP2, LEDP3, LEDP4, OUT1: (no value), pinhead:1X02
- added Q2: IRF530, transistor-power:TO220BV
- added R16: 1 M, resistor:0207/10
- added R17, R18, R21: 1k, resistor:0207/10
- added R19: 1.5k, resistor:0207/10
- added R20: 330, resistor:0207/10
- C1: value 4.7uF -> 100nF; device resistor:E2,5-6 -> resistor:C025-024X044
- C2: value 100nF -> 3.3 nF
- C3: value 100 nF -> 330 nF
- C5: value 3.3 nF -> 47 uF; device resistor:C025-024X044 -> rcl:E2,5-5
- C6: value 47 uF -> 10 uF
- C7: value 10 uF -> 4.7uF; device rcl:E2,5-5 -> resistor:E2,5-6
- IC1: value TL082P -> NE555N
- IC3: value NE555N -> 7805TV; device linear:DIL08 -> linear:TO220V
- R1: value 1M -> 470
- R10: value 4.7k -> 33
- R11: value 1k -> 33
- R12: value 150 -> 1M
- R13: value 470 -> 1k
- R14: value 330 -> 1k
- R15: value 1k -> 2.2 k
- R2: value 1k -> 470
- R3: value 1k -> 4.7k
- R4: value 2.2 k -> 1k
- R5: value 1 M -> 56k
- R6: value 1k -> 22k
- R7: value 1k -> 150
- R8: value 1.5k -> 33
- moved R9 110.9 mm to (-14.0, -24.1)
- moved R11 94.9 mm to (-14.0, -34.3), turned to 0 degrees
- moved R10 91.6 mm to (-14.0, -29.2), turned to 0 degrees
- moved R6 78.4 mm to (7.62, 7.62), turned to 270 degrees
- moved R7 68.6 mm to (6.35, 47.0), turned to 90 degrees
- moved R5 65.6 mm to (12.7, 7.62), turned to 270 degrees
- moved IC1 64.7 mm to (21.6, 7.62)
- moved C2 55.1 mm to (30.5, 6.35)
- moved R12 53.4 mm to (57.1, 63.5), turned to 0 degrees
- moved C7 52.2 mm to (47.0, 66.0)
- moved R2 47.9 mm to (16.5, 27.9), turned to 270 degrees
- moved R1 44.4 mm to (16.5, 45.7)
- moved C1 41.9 mm to (6.35, 55.9), turned to 90 degrees
- moved R13 40.7 mm to (57.1, 48.3)
- moved R3 34.9 mm to (22.9, 54.6), turned to 90 degrees
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- renumbered LED to LEDP1, PD to PD1
Connections:
- removed net N$33: C6.+, IC6.3
- removed net N$34: C5.1, IC6.2, IC6.6, R33.1
- removed net N$35: C6.-, D1.A, D2.C
- removed net VCC: C3.1, IC5.1
- new net LEDSIG: Q2.D, R10.1, R11.1, R13.1, R8.1, R9.1
- new net N$11: C5.-, D1.A, D2.C
- new net N$17: LEDP2.2, R9.2
- new net N$19: LEDP3.2, R10.2
- new net N$20: LEDP4.2, R11.2
- new net N$21: IC4.2, R14.2, R16.1
- new net VIN: C3.1, IC3.1, JP1.PWR
- net +5V: now also IC1.4, IC2.4, IC2.8, IC3.3, IC4.8, LEDP2.1, LEDP3.1, LEDP4.1, R12.2, R19.2, R21.2, R3.2, R5.2; no longer IC3.8, IC5.3, IC6.4, IC6.8, R1.2, R10.2, R15.2, R32.2, R8.2
- net -5V: now also C6.-, IC4.4; no longer C7.-, IC1.4
- net GND: now also C1.2, C6.+, C7.-, IC1.1, IC2.1, IC3.2, JP1.GND, JP1.GNDBREAK, OUT1.2, Q2.S, R1.1, R15.1, R18.1, R2.2; no longer C1.-, C5.2, C7.+, IC3.1, IC5.2, IC6.1, R13.1, R35.2, R4.1, R7.1, T1.3
- net N$1: now also C1.1, IC2.2, IC2.6, R4.1; no longer PD1.1, R1.1, R2.1
- net N$10: now also C5.+, IC1.3; no longer C2.1, IC3.2, IC3.6, R11.1
- net N$12: now also Q2.G, R7.2; no longer R12.2, T1.1
- net N$13: now also IC4.7, R20.2; no longer IC1.7, R14.2
- net N$14: now also R1.2; no longer R13.2
- net N$15: now also LEDP1.2, R8.2; no longer IC3.7, R10.1, R11.2
- net N$16: now also OUT1.1, R21.1; no longer OUT.1, R15.1
- net N$18: now also R20.1; no longer R14.1
- net N$2: now also IC2.7, R3.1, R4.2; no longer IC1.2, R2.2, R5.1
- net N$22: now also PD1.1, R12.1, R14.1; no longer R3.1, R9.1, T1.2
- net N$3: now also IC4.3, R13.2, R15.2; no longer IC1.3, R3.2, R4.2
- net N$32: now also R2.1; no longer R35.1
- net N$4: now also IC4.1, R16.2, R17.1; no longer IC1.1, R5.2, R6.1
- net N$5: now also C7.+, IC4.6, R17.2; no longer C1.+, IC1.6, R6.2
- net N$6: now also IC4.5, R18.2, R19.1; no longer IC1.5, R7.2, R8.1
- net N$7: now also C2.1, IC1.2, IC1.6, R6.1; no longer LEDP1.2, R9.2
- net N$8: now also IC1.7, R5.1, R6.2; no longer IC6.7, R32.1, R33.2
- net N$9: now also IC2.3, R7.1; no longer IC3.3, R12.1
